Commit message: Phase 4b: end-effector payload sweep (Exp 2 analog)
Adds a matching "payload" body/link to both the MJCF and URDF (mass from
one FR3_PAYLOAD_MASS_KG env var), fixing a real gap where a payload added
only to MuJoCo's model was invisible to B2/B3's certificate (fr3_dynamics
parses the URDF via kdl_parser, entirely independent of the MJCF).

run_experiment.py/compute_metrics.py refactored into reusable run_one()/
compute() functions plus a "large" goal choice, so the new
exp2_payload_sweep.py can drive many runs directly. Also fixes a real DDS
hang: "ros2 control load_controller" leaks a persistent per-domain-ID
ros2cli daemon on every launch, which a long sweep accumulates until the
transport wedges solid -- pkill_stragglers() now reaps those too.

Verified end-to-end: B3's certificate first triggers at 6kg payload, 4kg
before B2's own reactive intervention at 10kg, with min_margin trending
monotonically from 9.65 to -24.2 N*m across the swept range.

fr3.xml (previously entirely .gitignore'd as vendored Menagerie content)
is now force-added: the payload body is genuine platform-authored code,
not vendored, so it needs real version history like the local patches to
the other third-party trees do.

Co-Authored-By: Claude Sonnet 5 <noreply@anthropic.com>

File: fr3_mujoco_bringup/urdf/fr3_mujoco.urdf.xacro (robot description, xacro)
@@ -27,4 +27,33 @@
 <robot name="fr3" xmlns:xacro="http://www.ros.org/wiki/xacro">
   <xacro:include filename="$(find franka_description)/robots/fr3/fr3.urdf.xacro"/>
+  <!-- Phase 4b: end-effector payload. fr3_link8 (franka_description's own
+       virtual flange link, franka_robot.xacro) is at the SAME physical
+       offset MuJoCo's own attachment_site uses on fr3_link7 (both come
+       from Franka's own kinematics spec); attaching here with a zero
+       origin keeps both models' payload at the identical point.
+       This link's mass must genuinely be part of fr3_dynamics's own KDL
+       chain (root_link to tip_link) for B2/B3's certificate to see it at
+       all; adding the MJCF body alone (as an earlier pass in this phase
+       did) changes only the SIMULATED physics, not what the certificate
+       itself computes, since fr3_dynamics parses THIS URDF via
+       kdl_parser, entirely independently of the MJCF. b2.tip_link and
+       b3.tip_link must be set to "payload" (not "fr3_link8") for this
+       link's mass to actually enter the chain; see the b2/b3 config
+       YAMLs. 1e-6 kg is the same numerically-safe near-zero default
+       fr3.xml's own payload body and the Python reference's
+       Arm.set_payload_mass use, not a real physical claim. -->
+  <xacro:arg name="payload_mass" default="1e-6"/>
+  <link name="payload">
+    <inertial>
+      <mass value="$(arg payload_mass)"/>
+      <origin xyz="0 0 0" rpy="0 0 0"/>
+      <inertia ixx="1e-8" iyy="1e-8" izz="1e-8" ixy="0" ixz="0" iyz="0"/>
+    </inertial>
+  </link>
+  <joint name="payload_joint" type="fixed">
+    <parent link="fr3_link8"/>
+    <child link="payload"/>
+    <origin xyz="0 0 0" rpy="0 0 0"/>
+  </joint>
   <ros2_control name="MujocoSystem" type="system">
     <hardware>
